File: pcb_kicad/board.kicad_pcb (KiCad board)
At the start: 2 copper layers, 94 x 86 mm, 38 parts

Commit message: update file sturecture, add jlcnumber
Other:
- board text added: "JLCJLCJLCJLC"
Changed lines of the file:
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@@
 			(drillshape 0)
 			(scaleselection 1)
-			(outputdirectory "untitled_keyboard/")
+			(outputdirectory "../../MITOS_MK1_ks/pcb/")
 		)
 	)
@@
 		(layer "Edge.Cuts")
 	)
+	(gr_text "JLCJLCJLCJLC"
+		(at 234 185.25 0)
+		(layer "B.SilkS")
+		(effects
+			(font
+				(size 1 1)
+				(thickness 0.15)
+			)
+			(justify left bottom mirror)
+		)
+	)
 	(gr_text "MITOS\nB.JH"
