File: mk2_pcb/board.kicad_pcb (KiCad board)
At the start: 2 copper layers, 99 x 90 mm, 38 parts

Commit message: jlc mk2 update
Routing:
- net RAW: track 141.5 -> 149.8 mm
Other:
- board text added: "Design by xyz"
- board text added: "JLCJLCJLCJLC"
- board text added: "MITOS MK.2"
Changed lines of the file:
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@@
 			(outputformat 1)
 			(mirror no)
-			(drillshape 1)
+			(drillshape 0)
 			(scaleselection 1)
-			(outputdirectory "")
+			(outputdirectory "gbr/")
 		)
 	)
@@
 		(at 204.5 164.225 -90)
 		(property "Reference" "PWR1"
-			(at -3.6 0 360)
+			(at -3.6 0 0)
 			(layer "F.SilkS")
 			(hide yes)
@@
 		)
 		(fp_text user "PWR1"
-			(at -3.499998 0 360)
+			(at -3.499998 0 0)
 			(layer "B.SilkS")
 			(hide yes)
@@
 		(layer "Edge.Cuts")
 	)
+	(gr_text "Design by xyz"
+		(at 240.25 185.75 0)
+		(layer "B.SilkS")
+		(effects
+			(font
+				(size 1.5 1.5)
+				(thickness 0.25)
+				(bold yes)
+			)
+			(justify left bottom mirror)
+		)
+	)
+	(gr_text "MITOS\nMK.2"
+		(at 219.25 184.25 0)
+		(layer "B.SilkS")
+		(effects
+			(font
+				(size 4 4)
+				(thickness 0.3)
+				(bold yes)
+			)
+			(justify left bottom mirror)
+		)
+	)
+	(gr_text "MITOS\nMK.2"
+		(at 201.25 184.25 0)
+		(layer "F.SilkS")
+		(effects
+			(font
+				(size 4 4)
+				(thickness 0.3)
+				(bold yes)
+			)
+			(justify left bottom)
+		)
+	)
+	(gr_text "JLCJLCJLCJLC"
+		(at 224 186 0)
+		(layer "F.SilkS")
+		(effects
+			(font
+				(size 1.5 1.5)
+				(thickness 0.3)
+				(bold yes)
+			)
+			(justify left bottom)
+		)
+	)
 	(segment
 		(start 179.97 172.175)
@@
 	)
 	(segment
-		(start 203.825 180.156701)
-		(end 198.236701 185.745)
+		(start 169.323299 185.745)
+		(end 168.635 185.056701)
 		(width 0.25)
 		(layer "B.Cu")
@@
 	)
 	(segment
-		(start 203.825 162.565)
-		(end 203.825 180.156701)
+		(start 203.75 162.49)
+		(end 203.75 161.25)
 		(width 0.25)
 		(layer "B.Cu")
@@
 	)
 	(segment
-		(start 168.635 181.308308)
-		(end 169.593308 180.35)
+		(start 197 166)
+		(end 199 168)
 		(width 0.25)
 		(layer "B.Cu")
@@
 	)
 	(segment
-		(start 169.323299 185.745)
-		(end 168.635 185.056701)
+		(start 197.7 160.8)
+		(end 197 161.5)
+		(width 0.25)
+		(layer "B.Cu")
+		(net 28)
+	)
+	(segment
+		(start 199 184.981701)
+		(end 198.236701 185.745)
 		(width 0.25)
 		(layer "B.Cu")
@@
 	)
 	(segment
+		(start 203.3 160.8)
+		(end 197.7 160.8)
+		(width 0.25)
+		(layer "B.Cu")
+		(net 28)
+	)
+	(segment
 		(start 169.81 172.524695)
 		(end 169.085 173.249695)
@@
 	)
 	(segment
-		(start 203.75 162.49)
-		(end 203.825 162.565)
+		(start 197 161.5)
+		(end 197 166)
+		(width 0.25)
+		(layer "B.Cu")
+		(net 28)
+	)
+	(segment
+		(start 198.236701 185.745)
+		(end 169.323299 185.745)
 		(width 0.25)
 		(layer "B.Cu")
@@
 	)
 	(segment
-		(start 198.236701 185.745)
-		(end 169.323299 185.745)
+		(start 168.635 181.308308)
+		(end 169.593308 180.35)
 		(width 0.25)
 		(layer "B.Cu")
@@
 	)
 	(segment
+		(start 203.75 161.25)
+		(end 203.3 160.8)
+		(width 0.25)
+		(layer "B.Cu")
+		(net 28)
+	)
+	(segment
 		(start 169.085 173.850305)
 		(end 169.59 174.355305)
 		(width 0.25)
 		(layer "B.Cu")
+		(net 28)
+	)
+	(segment
+		(start 199 168)
+		(end 199 184.981701)
+		(width 0.25)
+		(layer "B.Cu")
