File: mitos_v3/pcbs/board.kicad_pcb (KiCad board)
At the start: 2 copper layers, 95.5 x 87 mm, 39 parts

Commit message: the real v3
Parts:
- added MH2: , ceoloide:mounting_hole_npth, F.Cu at (184.5, 160.8)
- added MH3: , ceoloide:mounting_hole_npth, F.Cu at (241.5, 121.9)
- added MH4: , ceoloide:mounting_hole_npth, F.Cu at (241.5, 179.8)
- CONN1: moved to F.Cu
- MCU1: footprint ceoloide:mcu_nice_nano -> ceoloide:mcu_supermini_nrf52840
- moved MH1 47.8 mm to (184.5, 119.9)
- moved CONN1 1.50 mm to (218.5, 161.0), turned to -90 degrees
- moved RST1 0.50 mm to (217.5, 184.0)
Routing:
- net P10: track 70.2 -> 98.1 mm
- net GND: track 121.8 -> 111.4 mm, vias 2 -> 1
- net P6: track 187.6 -> 196.7 mm
- net RAW: track 56.1 -> 49.8 mm
- net BAT_P: track 31.1 -> 27.7 mm, vias 3 -> 2
- net P4: track 124.5 -> 122.3 mm
- net inner_bottom: track 31.5 -> 30.0 mm
- net pinky_top: track 31.5 -> 30.0 mm
- net middle_bottom: track 31.4 -> 30.0 mm
- net inner_thumb: track 31.4 -> 30.0 mm
- net inner_home: track 31.4 -> 30.0 mm
- net index_thumb: track 31.4 -> 30.0 mm
- net index_home: track 31.4 -> 30.0 mm
- net index_bottom: track 31.4 -> 30.0 mm
- net ring_home: track 31.4 -> 30.0 mm
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